Commit message: Updated and verified robot model on Rviz

File: src/ur_robot_description/models/core.xacro (robot description, xacro)
@@ -1,50 +1,22 @@
 <?xml version="1.0"?>
 <robot xmlns:xacro="http://wiki.ros.org/xacro">
-  <xacro:include filename="$(find cobotizur_description)/models/include/arm.xacro"/>
-  <xacro:include filename="$(find cobotizur_description)/models/include/cobotizur.xacro"/>
-  <xacro:include filename="$(find cobotizur_description)/models/include/conveyor.xacro"/>
-  <xacro:include filename="$(find cobotizur_description)/models/include/tool.xacro"/>
-  <!-- parameters -->
-  <!-- possible 'mode' values: gz, hw -->
-  <xacro:arg name="mode" default=""/>
-  <!-- possible 'cobotizur_type' values: CT10, CF20 -->
-  <xacro:arg name="cobotizur_type" default="CX"/>
-  <xacro:property name="cobotizur_type" value="$(arg cobotizur_type)"/>
-  <!-- possible 'ur_type' values: ur3, ur3e, ur5, ur5e, ur7e, ur10, ur10e, ur12e, ur16e, ur15, ur20, ur30 -->
-  <xacro:property name="ur_type" value="urX"/>
-  <xacro:property name="ur_joint_xyz" value="0 0 0"/>
-  <xacro:property name="cb_joint_xyz" value="0 0 0"/>
-  <xacro:property name="conveyor_height" value="0"/>
-  <xacro:if value="${cobotizur_type == 'CT10'}">
-    <xacro:property name="ur_type" value="ur10"/>
-    <xacro:property name="ur_joint_xyz" value="0 0 0.97756792"/>
-    <xacro:property name="cb_joint_xyz" value="0 0.426 0.344"/>
-    <xacro:property name="conveyor_height" value="0.72"/>
-  </xacro:if>
-  <xacro:if value="${cobotizur_type == 'CF20'}">
-    <xacro:property name="ur_type" value="ur20"/>
-    <xacro:property name="ur_joint_xyz" value="0 0 1.4596"/>
-    <xacro:property name="cb_joint_xyz" value="0 0.426 0.344"/>
-    <xacro:property name="conveyor_height" value="1.08"/>
-  </xacro:if>
-  <xacro:macro name="robot_macro" params="mode cobotizur_type">
+  <xacro:include filename="$(find ur_robot_description)/models/include/arm.xacro"/>
+  <xacro:include filename="$(find ur_robot_description)/models/include/conveyor.xacro"/>
+  <xacro:include filename="$(find ur_robot_description)/models/include/tool.xacro"/>
+  <xacro:macro name="robot_macro" params="mode ur_type robot_ip simulation_controllers">
     <link name="unit"/>
     <xacro:conveyor_macro
-      height="${conveyor_height}"
-      parent="unit"
-    />
-    <xacro:cobotizur_macro
-      cobotizur_type="$(arg cobotizur_type)"
+      height="0.5"
       parent="unit"
     />
     <xacro:arm_macro
-      mode="$(arg mode)"
+      mode="${mode}"
       ur_type="${ur_type}"
-      parent="cobotizur"
-      arm_origin_xyz="${ur_joint_xyz}"
-      cb_origin_xyz="${cb_joint_xyz}"
+      parent="unit"
+      robot_ip="${robot_ip}"
+      simulation_controllers="${simulation_controllers}"
     />
     <xacro:tool_macro
-      cobotizur_type="$(arg cobotizur_type)"
+      mode="${mode}"
       parent="tool0"
     />

File: src/ur_robot_description/models/include/arm.xacro (robot description, xacro)
@@ -2,11 +2,5 @@
 <robot xmlns:xacro="http://wiki.ros.org/xacro">
   <xacro:include filename="$(find ur_description)/urdf/ur_macro.xacro"/>
-  <xacro:macro name="arm_macro" params="mode ur_type parent arm_origin_xyz cb_origin_xyz">
-    <xacro:if value="${mode == 'hw'}">
-      <xacro:property name="force_abs_paths" value="false"/>
-    </xacro:if>
-    <xacro:if value="${mode == 'gz' || mode == 'gazebo'}">
-      <xacro:property name="force_abs_paths" value="true"/>
-    </xacro:if>
+  <xacro:macro name="arm_macro" params="mode ur_type parent robot_ip simulation_controllers">
     <xacro:ur_robot
       name="ur"
@@ -17,11 +11,44 @@
       physical_parameters_file="$(find ur_description)/config/${ur_type}/physical_parameters.yaml"
       visual_parameters_file="$(find ur_description)/config/${ur_type}/visual_parameters.yaml"
+      transmission_hw_interface=""
       safety_limits="true"
       safety_pos_margin="0.15"
       safety_k_position="20"
-      force_abs_paths="${force_abs_paths}"
+      use_fake_hardware="false"
+      fake_sensor_commands="false"
+      sim_gazebo="false"
+      sim_ignition="${mode == 'gz'}"
+      headless_mode="true"
+      initial_positions="${dict(shoulder_pan_joint=0.0,shoulder_lift_joint=-1.57,elbow_joint=0.0,wrist_1_joint=-1.57,wrist_2_joint=0.0,wrist_3_joint=0.0)}"
+      use_tool_communication="false"
+      tool_voltage="0"
+      tool_parity="0"
+      tool_baud_rate="115200"
+      tool_stop_bits="1"
+      tool_rx_idle_chars="1.5"
+      tool_tx_idle_chars="3.5"
+      tool_device_name="/tmp/ttyUR"
+      tool_tcp_port="54321"
+      robot_ip="$(arg robot_ip)"
+      script_filename="$(find ur_robot_driver)/resources/ros_control.urscript"
+      output_recipe_filename="$(find ur_robot_driver)/resources/rtde_output_recipe.txt"
+      input_recipe_filename="$(find ur_robot_driver)/resources/rtde_input_recipe.txt"
+      reverse_ip="0.0.0.0"
+      reverse_port="50001"
+      script_sender_port="50002"
+      trajectory_port="50003"
+      script_command_port="50004"
     >
-      <origin xyz="${arm_origin_xyz}" rpy="0 0 0"/>
+      <origin xyz="0 0 0" rpy="0 0 0"/>          <!-- position robot in the world -->
     </xacro:ur_robot>
+    <xacro:if value="${mode == 'gz'}">
+      <gazebo reference="world"></gazebo>
+      <gazebo>
+        <plugin filename="libign_ros2_control-system.so" name="ign_ros2_control::IgnitionROS2ControlPlugin">
+          <parameters>$(arg simulation_controllers)</parameters>
+          <controller_manager_node_name>controller_manager</controller_manager_node_name>
+        </plugin>
+      </gazebo>
+    </xacro:if>
   </xacro:macro>
 </robot>

File: src/ur_robot_description/models/include/tool.xacro (robot description, xacro)
@@ -1,63 +1,15 @@
 <?xml version="1.0"?>
 <robot xmlns:xacro="http://wiki.ros.org/xacro">
-  <xacro:macro name="tool_macro" params="cobotizur_type parent">
-    <xacro:property name="tool_name" value=""/>
-    <xacro:property name="tool_origin_xyz" value="0 0 0"/>
-    <xacro:property name="tool_origin_rpy" value="0 0 0"/>
-    <xacro:property name="tool_collision" value="0 0 0"/>
-    <xacro:property name="tool_offset" value="0 0 0"/>
-    <xacro:if value="${cobotizur_type == 'CT10'}">
-      <xacro:property name="tool_name" value="VQ10"/>
-      <xacro:property name="tool_origin_xyz" value="0 0.175 0.13"/>
-      <xacro:property name="tool_origin_rpy" value="3.142 0 0"/>
-      <xacro:property name="tool_collision" value="0.313 0.34 0.16"/>
-      <xacro:property name="tool_offset" value="0 0.175 0.16"/>
-    </xacro:if>
-    <xacro:if value="${cobotizur_type == 'CF20'}">
-      <xacro:property name="tool_name" value="VQ20"/>
-      <xacro:property name="tool_origin_xyz" value="0 0 0.1398"/>
-      <xacro:property name="tool_origin_rpy" value="3.142 0 3.142"/>
-      <xacro:property name="tool_collision" value="0.36 0.185 0.1768"/>
-      <xacro:property name="tool_offset" value="0 0 0.1768"/>
-    </xacro:if>
-    <link name="tool">
-      <visual>
-        <origin xyz="${tool_origin_xyz}" rpy="${tool_origin_rpy}"/>
-        <geometry>
-          <mesh filename="file://$(find cobotizur_description)/models/meshes/tool/${tool_name}.stl"/>
-        </geometry>
-        <material name="white">
-          <color rgba="1 1 1 1"/>
-        </material>
-      </visual>
-      <collision>
-        <origin xyz="${tool_origin_xyz.split()[0]} ${float(tool_origin_xyz.split()[1])/2} ${float(tool_collision.split()[2])/2}" rpy="3.142 0 0"/>
-        <geometry>
-          <box size="${tool_collision}"/>
-        </geometry>
-      </collision>
-      <inertial>
-        <mass value="1"/>
-        <origin xyz="${tool_origin_xyz}" rpy="3.142 0 0"/>
-        <inertia ixx="0.01" ixy="0.0" ixz="0.0" iyy="0.01" iyz="0.0" izz="0.01"/>
-      </inertial>
-    </link>
-    <joint name="tool_joint" type="fixed">
-      <origin xyz="0 0 0" rpy="0 0 3.142"/>
-      <parent link="${parent}"/>
-      <child link="tool"/>
-    </joint>
-    <link name="vacuum_pad"/>
-    <joint name="vacuum_pad_joint" type="fixed">
-      <origin xyz="${tool_offset}" rpy="0 0 0"/>
-      <parent link="tool"/>
-      <child link="vacuum_pad"/>
-    </joint>
-    <link name="vacuum_pad0"/>
-    <joint name="vacuum_pad0_joint" type="fixed">
+  <xacro:include filename="$(find robotiq_description)/urdf/robotiq_2f_85_macro.urdf.xacro" />
+  <xacro:macro name="tool_macro" params="mode parent">
+    <xacro:robotiq_gripper
+      name="RobotiqGripperHardwareInterface"
+      prefix=""
+      parent="${parent}"
+      sim_ignition="${mode == 'gz'}"
+      include_ros2_control="false"
+    >
       <origin xyz="0 0 0" rpy="0 0 0"/>
-      <parent link="vacuum_pad"/>
-      <child link="vacuum_pad0"/>
-    </joint>
+    </xacro:robotiq_gripper>
   </xacro:macro>
 </robot>

File: src/ur_robot_description/models/robot.urdf.xacro (robot description, xacro)
@@ -1,13 +1,17 @@
 <?xml version="1.0"?>
 <robot xmlns:xacro="http://wiki.ros.org/xacro" name="robot">
-  <xacro:include filename="$(find cobotizur_description)/models/core.xacro"/>
+  <xacro:include filename="$(find ur_robot_description)/models/core.xacro"/>
   <!-- parameters -->
   <!-- possible 'mode' values: gz, hw -->
   <xacro:arg name="mode" default=""/>
-  <!-- possible 'cobotizur_type' values: CT10, CF20 -->
-  <xacro:arg name="cobotizur_type" default="CX"/>
+  <!-- possible 'ur_type' values: ur3, ur5, ur10, ur3e, ur5e, ur7e, ur10e, ur12e, ur16e, ur8long, ur15, ur18, ur20, ur30 -->
+  <xacro:arg name="ur_type" default="urX"/>
+  <xacro:arg name="robot_ip" default="0.0.0.0"/>
+  <xacro:arg name="simulation_controllers" default=""/>
   <xacro:robot_macro
     mode="$(arg mode)"
-    cobotizur_type="$(arg cobotizur_type)"
+    ur_type="$(arg ur_type)"
+    robot_ip="$(arg robot_ip)"
+    simulation_controllers="$(arg simulation_controllers)"
   />
 </robot>
